Commit message: Add assembly eval pipeline: trajectories, env URDFs, and eval_assembly.py
- Rewrite generate_trajectories.py to sample crane-style waypoints from
  evaluate_trajectory() and generate per-sub-problem environment URDFs
  with completed parts baked in as static geometry
- Rewrite objects.py to auto-load canonical extents from
  canonical_transforms.json and create URDFs referencing canonical meshes
- Create eval_assembly.py for sequential sub-problem evaluation
- Generate pick_place trajectories and environment URDFs for all assemblies

Co-Authored-By: Claude Opus 4.6 <noreply@anthropic.com>

File: assets/urdf/fabrica/beam/0/beam_0.urdf (robot description, URDF)
Before this commit: robot beam_0, 1 links, 0 joints
Links:
- link beam_0: geometry collision mesh filename=0_canonical.obj scale=1 1 1; visual mesh filename=0_canonical.obj scale=1 1 1

File: assets/urdf/fabrica/beam/1/beam_1.urdf (robot description, URDF)
Before this commit: robot beam_1, 1 links, 0 joints
Links:
- link beam_1: geometry collision mesh filename=1_canonical.obj scale=1 1 1; visual mesh filename=1_canonical.obj scale=1 1 1

File: assets/urdf/fabrica/beam/2/beam_2.urdf (robot description, URDF)
Before this commit: robot beam_2, 1 links, 0 joints
Links:
- link beam_2: geometry collision mesh filename=2_canonical.obj scale=1 1 1; visual mesh filename=2_canonical.obj scale=1 1 1

File: assets/urdf/fabrica/beam/3/beam_3.urdf (robot description, URDF)
Before this commit: robot beam_3, 1 links, 0 joints
Links:
- link beam_3: geometry collision mesh filename=3_canonical.obj scale=1 1 1; visual mesh filename=3_canonical.obj scale=1 1 1

File: assets/urdf/fabrica/beam/6/beam_6.urdf (robot description, URDF)
Before this commit: robot beam_6, 1 links, 0 joints
Links:
- link beam_6: geometry collision mesh filename=6_canonical.obj scale=1 1 1; visual mesh filename=6_canonical.obj scale=1 1 1

File: assets/urdf/fabrica/car/0/car_0.urdf (robot description, URDF)
Before this commit: robot car_0, 1 links, 0 joints
Links:
- link car_0: geometry collision mesh filename=0_canonical.obj scale=1 1 1; visual mesh filename=0_canonical.obj scale=1 1 1

File: assets/urdf/fabrica/car/1/car_1.urdf (robot description, URDF)
Before this commit: robot car_1, 1 links, 0 joints
Links:
- link car_1: geometry collision mesh filename=1_canonical.obj scale=1 1 1; visual mesh filename=1_canonical.obj scale=1 1 1

File: assets/urdf/fabrica/car/2/car_2.urdf (robot description, URDF)
Before this commit: robot car_2, 1 links, 0 joints
Links:
- link car_2: geometry collision mesh filename=2_canonical.obj scale=1 1 1; visual mesh filename=2_canonical.obj scale=1 1 1

File: assets/urdf/fabrica/car/3/car_3.urdf (robot description, URDF)
Before this commit: robot car_3, 1 links, 0 joints
Links:
- link car_3: geometry collision mesh filename=3_canonical.obj scale=1 1 1; visual mesh filename=3_canonical.obj scale=1 1 1

File: assets/urdf/fabrica/car/4/car_4.urdf (robot description, URDF)
Before this commit: robot car_4, 1 links, 0 joints
Links:
- link car_4: geometry collision mesh filename=4_canonical.obj scale=1 1 1; visual mesh filename=4_canonical.obj scale=1 1 1

File: assets/urdf/fabrica/car/5/car_5.urdf (robot description, URDF)
Before this commit: robot car_5, 1 links, 0 joints
Links:
- link car_5: geometry collision mesh filename=5_canonical.obj scale=1 1 1; visual mesh filename=5_canonical.obj scale=1 1 1

File: assets/urdf/fabrica/cooling_manifold/0/cooling_manifold_0.urdf (robot description, URDF)
Before this commit: robot cooling_manifold_0, 1 links, 0 joints
Links:
- link cooling_manifold_0: geometry collision mesh filename=0_canonical.obj scale=1 1 1; visual mesh filename=0_canonical.obj scale=1 1 1

File: assets/urdf/fabrica/cooling_manifold/1/cooling_manifold_1.urdf (robot description, URDF)
Before this commit: robot cooling_manifold_1, 1 links, 0 joints
Links:
- link cooling_manifold_1: geometry collision mesh filename=1_canonical.obj scale=1 1 1; visual mesh filename=1_canonical.obj scale=1 1 1

File: assets/urdf/fabrica/cooling_manifold/2/cooling_manifold_2.urdf (robot description, URDF)
Before this commit: robot cooling_manifold_2, 1 links, 0 joints
Links:
- link cooling_manifold_2: geometry collision mesh filename=2_canonical.obj scale=1 1 1; visual mesh filename=2_canonical.obj scale=1 1 1

File: assets/urdf/fabrica/cooling_manifold/3/cooling_manifold_3.urdf (robot description, URDF)
Before this commit: robot cooling_manifold_3, 1 links, 0 joints
Links:
- link cooling_manifold_3: geometry collision mesh filename=3_canonical.obj scale=1 1 1; visual mesh filename=3_canonical.obj scale=1 1 1

File: assets/urdf/fabrica/cooling_manifold/4/cooling_manifold_4.urdf (robot description, URDF)
Before this commit: robot cooling_manifold_4, 1 links, 0 joints
Links:
- link cooling_manifold_4: geometry collision mesh filename=4_canonical.obj scale=1 1 1; visual mesh filename=4_canonical.obj scale=1 1 1

File: assets/urdf/fabrica/cooling_manifold/5/cooling_manifold_5.urdf (robot description, URDF)
Before this commit: robot cooling_manifold_5, 1 links, 0 joints
Links:
- link cooling_manifold_5: geometry collision mesh filename=5_canonical.obj scale=1 1 1; visual mesh filename=5_canonical.obj scale=1 1 1

File: assets/urdf/fabrica/cooling_manifold/6/cooling_manifold_6.urdf (robot description, URDF)
Before this commit: robot cooling_manifold_6, 1 links, 0 joints
Links:
- link cooling_manifold_6: geometry collision mesh filename=6_canonical.obj scale=1 1 1; visual mesh filename=6_canonical.obj scale=1 1 1

File: assets/urdf/fabrica/duct/0/duct_0.urdf (robot description, URDF)
Before this commit: robot duct_0, 1 links, 0 joints
Links:
- link duct_0: geometry collision mesh filename=0_canonical.obj scale=1 1 1; visual mesh filename=0_canonical.obj scale=1 1 1

File: assets/urdf/fabrica/duct/1/duct_1.urdf (robot description, URDF)
Before this commit: robot duct_1, 1 links, 0 joints
Links:
- link duct_1: geometry collision mesh filename=1_canonical.obj scale=1 1 1; visual mesh filename=1_canonical.obj scale=1 1 1
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