Commit message: Add CoACD collision meshes, environment URDFs, and debug/eval scripts
Co-Authored-By: Claude Opus 4.6 (1M context) <noreply@anthropic.com>

File: assets/urdf/fabrica/environments/beam_0/scene_sdf.urdf (robot description, URDF)
Before this commit: robot table_beam_2_scene_sdf, 2 links, 1 joints
Links:
- added link part_2; collision mesh filename=../../beam/2/2_canonical.obj scale=1 1 1; visual mesh filename=../../beam/2/2_canonical.obj scale=1 1 1
Joints:
- added joint part_2_joint: type fixed, parent box, child part_2, origin xyz=-0.124463 0.04 0.18810000000000004 rpy=3.141592653589793 -1.5707963267948966 3.141592653589793
