Commit message: Fix scene URDF gimbal lock bug, add viser rotation, cleanup
- Fix quaternion-to-RPY gimbal lock in generate_table_urdfs.py: hand-rolled
  conversion produced (180°,-90°,180°) instead of (0°,-90°,0°) — a different
  rotation entirely. Now uses scipy. Regenerated all beam scene URDFs.
- Fix viser_viz.py: _load_scene_urdf() was ignoring joint rotation, only
  applying translation. Now extracts full quaternion from origin matrix.
- Delete all unused pick_place.urdf files (46 files, unreferenced dead code)
- Add validate_scenes.py for visual inspection of scene URDFs + trajectories
- Update CLAUDE.md: don't kill ports blindly

Co-Authored-By: Claude Opus 4.6 (1M context) <noreply@anthropic.com>

File: assets/urdf/fabrica/environments/beam_0/scene.urdf (robot description, URDF)
Before this commit: robot table_beam_0_scene, 3 links, 2 joints
Joints:
- joint part_2_joint: origin xyz=-0.124463 0.04 0.18810000000000004 rpy=3.141592653589793 -1.5707963267948966 3.141592653589793 -> xyz=-0.124463 0.04 0.18810000000000004 rpy=0.0 -1.5707963057214722 0.0
- joint part_6_joint: origin xyz=-0.08 0.04 0.15674100000000002 rpy=0.0 -0.0 0.0 -> xyz=-0.08 0.04 0.15674100000000002 rpy=0.0 0.0 0.0

File: assets/urdf/fabrica/environments/beam_0/scene_coacd.urdf (robot description, URDF)
Before this commit: robot table_beam_0_scene_coacd, 34 links, 33 joints
Joints:
- joint part_2_hull_0_joint: origin xyz=-0.124463 0.04 0.18810000000000004 rpy=3.141592653589793 -1.5707963267948966 3.141592653589793 -> xyz=-0.124463 0.04 0.18810000000000004 rpy=0.0 -1.5707963057214722 0.0
- joint part_2_hull_10_joint: origin xyz=-0.124463 0.04 0.18810000000000004 rpy=3.141592653589793 -1.5707963267948966 3.141592653589793 -> xyz=-0.124463 0.04 0.18810000000000004 rpy=0.0 -1.5707963057214722 0.0
- joint part_2_hull_11_joint: origin xyz=-0.124463 0.04 0.18810000000000004 rpy=3.141592653589793 -1.5707963267948966 3.141592653589793 -> xyz=-0.124463 0.04 0.18810000000000004 rpy=0.0 -1.5707963057214722 0.0
- joint part_2_hull_12_joint: origin xyz=-0.124463 0.04 0.18810000000000004 rpy=3.141592653589793 -1.5707963267948966 3.141592653589793 -> xyz=-0.124463 0.04 0.18810000000000004 rpy=0.0 -1.5707963057214722 0.0
- joint part_2_hull_13_joint: origin xyz=-0.124463 0.04 0.18810000000000004 rpy=3.141592653589793 -1.5707963267948966 3.141592653589793 -> xyz=-0.124463 0.04 0.18810000000000004 rpy=0.0 -1.5707963057214722 0.0
- joint part_2_hull_14_joint: origin xyz=-0.124463 0.04 0.18810000000000004 rpy=3.141592653589793 -1.5707963267948966 3.141592653589793 -> xyz=-0.124463 0.04 0.18810000000000004 rpy=0.0 -1.5707963057214722 0.0
- joint part_2_hull_15_joint: origin xyz=-0.124463 0.04 0.18810000000000004 rpy=3.141592653589793 -1.5707963267948966 3.141592653589793 -> xyz=-0.124463 0.04 0.18810000000000004 rpy=0.0 -1.5707963057214722 0.0
- joint part_2_hull_16_joint: origin xyz=-0.124463 0.04 0.18810000000000004 rpy=3.141592653589793 -1.5707963267948966 3.141592653589793 -> xyz=-0.124463 0.04 0.18810000000000004 rpy=0.0 -1.5707963057214722 0.0
- joint part_2_hull_17_joint: origin xyz=-0.124463 0.04 0.18810000000000004 rpy=3.141592653589793 -1.5707963267948966 3.141592653589793 -> xyz=-0.124463 0.04 0.18810000000000004 rpy=0.0 -1.5707963057214722 0.0
- joint part_2_hull_1_joint: origin xyz=-0.124463 0.04 0.18810000000000004 rpy=3.141592653589793 -1.5707963267948966 3.141592653589793 -> xyz=-0.124463 0.04 0.18810000000000004 rpy=0.0 -1.5707963057214722 0.0
- joint part_2_hull_2_joint: origin xyz=-0.124463 0.04 0.18810000000000004 rpy=3.141592653589793 -1.5707963267948966 3.141592653589793 -> xyz=-0.124463 0.04 0.18810000000000004 rpy=0.0 -1.5707963057214722 0.0
- joint part_2_hull_3_joint: origin xyz=-0.124463 0.04 0.18810000000000004 rpy=3.141592653589793 -1.5707963267948966 3.141592653589793 -> xyz=-0.124463 0.04 0.18810000000000004 rpy=0.0 -1.5707963057214722 0.0
- joint part_2_hull_4_joint: origin xyz=-0.124463 0.04 0.18810000000000004 rpy=3.141592653589793 -1.5707963267948966 3.141592653589793 -> xyz=-0.124463 0.04 0.18810000000000004 rpy=0.0 -1.5707963057214722 0.0
- joint part_2_hull_5_joint: origin xyz=-0.124463 0.04 0.18810000000000004 rpy=3.141592653589793 -1.5707963267948966 3.141592653589793 -> xyz=-0.124463 0.04 0.18810000000000004 rpy=0.0 -1.5707963057214722 0.0
- joint part_2_hull_6_joint: origin xyz=-0.124463 0.04 0.18810000000000004 rpy=3.141592653589793 -1.5707963267948966 3.141592653589793 -> xyz=-0.124463 0.04 0.18810000000000004 rpy=0.0 -1.5707963057214722 0.0
- joint part_2_hull_7_joint: origin xyz=-0.124463 0.04 0.18810000000000004 rpy=3.141592653589793 -1.5707963267948966 3.141592653589793 -> xyz=-0.124463 0.04 0.18810000000000004 rpy=0.0 -1.5707963057214722 0.0
- joint part_2_hull_8_joint: origin xyz=-0.124463 0.04 0.18810000000000004 rpy=3.141592653589793 -1.5707963267948966 3.141592653589793 -> xyz=-0.124463 0.04 0.18810000000000004 rpy=0.0 -1.5707963057214722 0.0
- joint part_2_hull_9_joint: origin xyz=-0.124463 0.04 0.18810000000000004 rpy=3.141592653589793 -1.5707963267948966 3.141592653589793 -> xyz=-0.124463 0.04 0.18810000000000004 rpy=0.0 -1.5707963057214722 0.0
- joint part_6_hull_0_joint: origin xyz=-0.08 0.04 0.15674100000000002 rpy=0.0 -0.0 0.0 -> xyz=-0.08 0.04 0.15674100000000002 rpy=0.0 0.0 0.0
- joint part_6_hull_10_joint: origin xyz=-0.08 0.04 0.15674100000000002 rpy=0.0 -0.0 0.0 -> xyz=-0.08 0.04 0.15674100000000002 rpy=0.0 0.0 0.0
- joint part_6_hull_11_joint: origin xyz=-0.08 0.04 0.15674100000000002 rpy=0.0 -0.0 0.0 -> xyz=-0.08 0.04 0.15674100000000002 rpy=0.0 0.0 0.0
- joint part_6_hull_12_joint: origin xyz=-0.08 0.04 0.15674100000000002 rpy=0.0 -0.0 0.0 -> xyz=-0.08 0.04 0.15674100000000002 rpy=0.0 0.0 0.0
- joint part_6_hull_13_joint: origin xyz=-0.08 0.04 0.15674100000000002 rpy=0.0 -0.0 0.0 -> xyz=-0.08 0.04 0.15674100000000002 rpy=0.0 0.0 0.0
- joint part_6_hull_14_joint: origin xyz=-0.08 0.04 0.15674100000000002 rpy=0.0 -0.0 0.0 -> xyz=-0.08 0.04 0.15674100000000002 rpy=0.0 0.0 0.0
- joint part_6_hull_1_joint: origin xyz=-0.08 0.04 0.15674100000000002 rpy=0.0 -0.0 0.0 -> xyz=-0.08 0.04 0.15674100000000002 rpy=0.0 0.0 0.0
- joint part_6_hull_2_joint: origin xyz=-0.08 0.04 0.15674100000000002 rpy=0.0 -0.0 0.0 -> xyz=-0.08 0.04 0.15674100000000002 rpy=0.0 0.0 0.0
- joint part_6_hull_3_joint: origin xyz=-0.08 0.04 0.15674100000000002 rpy=0.0 -0.0 0.0 -> xyz=-0.08 0.04 0.15674100000000002 rpy=0.0 0.0 0.0
- joint part_6_hull_4_joint: origin xyz=-0.08 0.04 0.15674100000000002 rpy=0.0 -0.0 0.0 -> xyz=-0.08 0.04 0.15674100000000002 rpy=0.0 0.0 0.0
- joint part_6_hull_5_joint: origin xyz=-0.08 0.04 0.15674100000000002 rpy=0.0 -0.0 0.0 -> xyz=-0.08 0.04 0.15674100000000002 rpy=0.0 0.0 0.0
- joint part_6_hull_6_joint: origin xyz=-0.08 0.04 0.15674100000000002 rpy=0.0 -0.0 0.0 -> xyz=-0.08 0.04 0.15674100000000002 rpy=0.0 0.0 0.0
- joint part_6_hull_7_joint: origin xyz=-0.08 0.04 0.15674100000000002 rpy=0.0 -0.0 0.0 -> xyz=-0.08 0.04 0.15674100000000002 rpy=0.0 0.0 0.0
- joint part_6_hull_8_joint: origin xyz=-0.08 0.04 0.15674100000000002 rpy=0.0 -0.0 0.0 -> xyz=-0.08 0.04 0.15674100000000002 rpy=0.0 0.0 0.0
- joint part_6_hull_9_joint: origin xyz=-0.08 0.04 0.15674100000000002 rpy=0.0 -0.0 0.0 -> xyz=-0.08 0.04 0.15674100000000002 rpy=0.0 0.0 0.0

File: assets/urdf/fabrica/environments/beam_0/scene_sdf.urdf (robot description, URDF)
Before this commit: robot table_beam_0_scene_sdf, 3 links, 2 joints
Joints:
- joint part_2_joint: origin xyz=-0.124463 0.04 0.18810000000000004 rpy=3.141592653589793 -1.5707963267948966 3.141592653589793 -> xyz=-0.124463 0.04 0.18810000000000004 rpy=0.0 -1.5707963057214722 0.0
- joint part_6_joint: origin xyz=-0.08 0.04 0.15674100000000002 rpy=0.0 -0.0 0.0 -> xyz=-0.08 0.04 0.15674100000000002 rpy=0.0 0.0 0.0

File: assets/urdf/fabrica/environments/beam_1/scene.urdf (robot description, URDF)
Before this commit: robot table_beam_1_scene, 5 links, 4 joints
Joints:
- joint part_2_joint: origin xyz=-0.124463 0.04 0.18810000000000004 rpy=3.141592653589793 -1.5707963267948966 3.141592653589793 -> xyz=-0.124463 0.04 0.18810000000000004 rpy=0.0 -1.5707963057214722 0.0
- joint part_3_joint: origin xyz=-0.035537 0.04 0.18810000000000004 rpy=3.141592653589793 -1.5707963267948966 3.141592653589793 -> xyz=-0.035537 0.04 0.18810000000000004 rpy=0.0 -1.5707963057214722 0.0
- joint part_6_joint: origin xyz=-0.08 0.04 0.15674100000000002 rpy=0.0 -0.0 0.0 -> xyz=-0.08 0.04 0.15674100000000002 rpy=0.0 0.0 0.0

File: assets/urdf/fabrica/environments/beam_1/scene_coacd.urdf (robot description, URDF)
Before this commit: robot table_beam_1_scene_coacd, 59 links, 58 joints
Joints:
- joint part_2_hull_0_joint: origin xyz=-0.124463 0.04 0.18810000000000004 rpy=3.141592653589793 -1.5707963267948966 3.141592653589793 -> xyz=-0.124463 0.04 0.18810000000000004 rpy=0.0 -1.5707963057214722 0.0
- joint part_2_hull_10_joint: origin xyz=-0.124463 0.04 0.18810000000000004 rpy=3.141592653589793 -1.5707963267948966 3.141592653589793 -> xyz=-0.124463 0.04 0.18810000000000004 rpy=0.0 -1.5707963057214722 0.0
- joint part_2_hull_11_joint: origin xyz=-0.124463 0.04 0.18810000000000004 rpy=3.141592653589793 -1.5707963267948966 3.141592653589793 -> xyz=-0.124463 0.04 0.18810000000000004 rpy=0.0 -1.5707963057214722 0.0
- joint part_2_hull_12_joint: origin xyz=-0.124463 0.04 0.18810000000000004 rpy=3.141592653589793 -1.5707963267948966 3.141592653589793 -> xyz=-0.124463 0.04 0.18810000000000004 rpy=0.0 -1.5707963057214722 0.0
- joint part_2_hull_13_joint: origin xyz=-0.124463 0.04 0.18810000000000004 rpy=3.141592653589793 -1.5707963267948966 3.141592653589793 -> xyz=-0.124463 0.04 0.18810000000000004 rpy=0.0 -1.5707963057214722 0.0
- joint part_2_hull_14_joint: origin xyz=-0.124463 0.04 0.18810000000000004 rpy=3.141592653589793 -1.5707963267948966 3.141592653589793 -> xyz=-0.124463 0.04 0.18810000000000004 rpy=0.0 -1.5707963057214722 0.0
- joint part_2_hull_15_joint: origin xyz=-0.124463 0.04 0.18810000000000004 rpy=3.141592653589793 -1.5707963267948966 3.141592653589793 -> xyz=-0.124463 0.04 0.18810000000000004 rpy=0.0 -1.5707963057214722 0.0
- joint part_2_hull_16_joint: origin xyz=-0.124463 0.04 0.18810000000000004 rpy=3.141592653589793 -1.5707963267948966 3.141592653589793 -> xyz=-0.124463 0.04 0.18810000000000004 rpy=0.0 -1.5707963057214722 0.0
- joint part_2_hull_17_joint: origin xyz=-0.124463 0.04 0.18810000000000004 rpy=3.141592653589793 -1.5707963267948966 3.141592653589793 -> xyz=-0.124463 0.04 0.18810000000000004 rpy=0.0 -1.5707963057214722 0.0
- joint part_2_hull_1_joint: origin xyz=-0.124463 0.04 0.18810000000000004 rpy=3.141592653589793 -1.5707963267948966 3.141592653589793 -> xyz=-0.124463 0.04 0.18810000000000004 rpy=0.0 -1.5707963057214722 0.0
- joint part_2_hull_2_joint: origin xyz=-0.124463 0.04 0.18810000000000004 rpy=3.141592653589793 -1.5707963267948966 3.141592653589793 -> xyz=-0.124463 0.04 0.18810000000000004 rpy=0.0 -1.5707963057214722 0.0
- joint part_2_hull_3_joint: origin xyz=-0.124463 0.04 0.18810000000000004 rpy=3.141592653589793 -1.5707963267948966 3.141592653589793 -> xyz=-0.124463 0.04 0.18810000000000004 rpy=0.0 -1.5707963057214722 0.0
- joint part_2_hull_4_joint: origin xyz=-0.124463 0.04 0.18810000000000004 rpy=3.141592653589793 -1.5707963267948966 3.141592653589793 -> xyz=-0.124463 0.04 0.18810000000000004 rpy=0.0 -1.5707963057214722 0.0
- joint part_2_hull_5_joint: origin xyz=-0.124463 0.04 0.18810000000000004 rpy=3.141592653589793 -1.5707963267948966 3.141592653589793 -> xyz=-0.124463 0.04 0.18810000000000004 rpy=0.0 -1.5707963057214722 0.0
- joint part_2_hull_6_joint: origin xyz=-0.124463 0.04 0.18810000000000004 rpy=3.141592653589793 -1.5707963267948966 3.141592653589793 -> xyz=-0.124463 0.04 0.18810000000000004 rpy=0.0 -1.5707963057214722 0.0
- joint part_2_hull_7_joint: origin xyz=-0.124463 0.04 0.18810000000000004 rpy=3.141592653589793 -1.5707963267948966 3.141592653589793 -> xyz=-0.124463 0.04 0.18810000000000004 rpy=0.0 -1.5707963057214722 0.0
- joint part_2_hull_8_joint: origin xyz=-0.124463 0.04 0.18810000000000004 rpy=3.141592653589793 -1.5707963267948966 3.141592653589793 -> xyz=-0.124463 0.04 0.18810000000000004 rpy=0.0 -1.5707963057214722 0.0
- joint part_2_hull_9_joint: origin xyz=-0.124463 0.04 0.18810000000000004 rpy=3.141592653589793 -1.5707963267948966 3.141592653589793 -> xyz=-0.124463 0.04 0.18810000000000004 rpy=0.0 -1.5707963057214722 0.0
- joint part_3_hull_0_joint: origin xyz=-0.035537 0.04 0.18810000000000004 rpy=3.141592653589793 -1.5707963267948966 3.141592653589793 -> xyz=-0.035537 0.04 0.18810000000000004 rpy=0.0 -1.5707963057214722 0.0
- joint part_3_hull_10_joint: origin xyz=-0.035537 0.04 0.18810000000000004 rpy=3.141592653589793 -1.5707963267948966 3.141592653589793 -> xyz=-0.035537 0.04 0.18810000000000004 rpy=0.0 -1.5707963057214722 0.0
- joint part_3_hull_11_joint: origin xyz=-0.035537 0.04 0.18810000000000004 rpy=3.141592653589793 -1.5707963267948966 3.141592653589793 -> xyz=-0.035537 0.04 0.18810000000000004 rpy=0.0 -1.5707963057214722 0.0
- joint part_3_hull_12_joint: origin xyz=-0.035537 0.04 0.18810000000000004 rpy=3.141592653589793 -1.5707963267948966 3.141592653589793 -> xyz=-0.035537 0.04 0.18810000000000004 rpy=0.0 -1.5707963057214722 0.0
- joint part_3_hull_13_joint: origin xyz=-0.035537 0.04 0.18810000000000004 rpy=3.141592653589793 -1.5707963267948966 3.141592653589793 -> xyz=-0.035537 0.04 0.18810000000000004 rpy=0.0 -1.5707963057214722 0.0
- joint part_3_hull_14_joint: origin xyz=-0.035537 0.04 0.18810000000000004 rpy=3.141592653589793 -1.5707963267948966 3.141592653589793 -> xyz=-0.035537 0.04 0.18810000000000004 rpy=0.0 -1.5707963057214722 0.0
- joint part_3_hull_15_joint: origin xyz=-0.035537 0.04 0.18810000000000004 rpy=3.141592653589793 -1.5707963267948966 3.141592653589793 -> xyz=-0.035537 0.04 0.18810000000000004 rpy=0.0 -1.5707963057214722 0.0
- joint part_3_hull_16_joint: origin xyz=-0.035537 0.04 0.18810000000000004 rpy=3.141592653589793 -1.5707963267948966 3.141592653589793 -> xyz=-0.035537 0.04 0.18810000000000004 rpy=0.0 -1.5707963057214722 0.0
- joint part_3_hull_1_joint: origin xyz=-0.035537 0.04 0.18810000000000004 rpy=3.141592653589793 -1.5707963267948966 3.141592653589793 -> xyz=-0.035537 0.04 0.18810000000000004 rpy=0.0 -1.5707963057214722 0.0
- joint part_3_hull_2_joint: origin xyz=-0.035537 0.04 0.18810000000000004 rpy=3.141592653589793 -1.5707963267948966 3.141592653589793 -> xyz=-0.035537 0.04 0.18810000000000004 rpy=0.0 -1.5707963057214722 0.0
- joint part_3_hull_3_joint: origin xyz=-0.035537 0.04 0.18810000000000004 rpy=3.141592653589793 -1.5707963267948966 3.141592653589793 -> xyz=-0.035537 0.04 0.18810000000000004 rpy=0.0 -1.5707963057214722 0.0
- joint part_3_hull_4_joint: origin xyz=-0.035537 0.04 0.18810000000000004 rpy=3.141592653589793 -1.5707963267948966 3.141592653589793 -> xyz=-0.035537 0.04 0.18810000000000004 rpy=0.0 -1.5707963057214722 0.0
- joint part_3_hull_5_joint: origin xyz=-0.035537 0.04 0.18810000000000004 rpy=3.141592653589793 -1.5707963267948966 3.141592653589793 -> xyz=-0.035537 0.04 0.18810000000000004 rpy=0.0 -1.5707963057214722 0.0
- joint part_3_hull_6_joint: origin xyz=-0.035537 0.04 0.18810000000000004 rpy=3.141592653589793 -1.5707963267948966 3.141592653589793 -> xyz=-0.035537 0.04 0.18810000000000004 rpy=0.0 -1.5707963057214722 0.0
- joint part_3_hull_7_joint: origin xyz=-0.035537 0.04 0.18810000000000004 rpy=3.141592653589793 -1.5707963267948966 3.141592653589793 -> xyz=-0.035537 0.04 0.18810000000000004 rpy=0.0 -1.5707963057214722 0.0
- joint part_3_hull_8_joint: origin xyz=-0.035537 0.04 0.18810000000000004 rpy=3.141592653589793 -1.5707963267948966 3.141592653589793 -> xyz=-0.035537 0.04 0.18810000000000004 rpy=0.0 -1.5707963057214722 0.0
- joint part_3_hull_9_joint: origin xyz=-0.035537 0.04 0.18810000000000004 rpy=3.141592653589793 -1.5707963267948966 3.141592653589793 -> xyz=-0.035537 0.04 0.18810000000000004 rpy=0.0 -1.5707963057214722 0.0
- joint part_6_hull_0_joint: origin xyz=-0.08 0.04 0.15674100000000002 rpy=0.0 -0.0 0.0 -> xyz=-0.08 0.04 0.15674100000000002 rpy=0.0 0.0 0.0
- joint part_6_hull_10_joint: origin xyz=-0.08 0.04 0.15674100000000002 rpy=0.0 -0.0 0.0 -> xyz=-0.08 0.04 0.15674100000000002 rpy=0.0 0.0 0.0
- joint part_6_hull_11_joint: origin xyz=-0.08 0.04 0.15674100000000002 rpy=0.0 -0.0 0.0 -> xyz=-0.08 0.04 0.15674100000000002 rpy=0.0 0.0 0.0
- joint part_6_hull_12_joint: origin xyz=-0.08 0.04 0.15674100000000002 rpy=0.0 -0.0 0.0 -> xyz=-0.08 0.04 0.15674100000000002 rpy=0.0 0.0 0.0
- joint part_6_hull_13_joint: origin xyz=-0.08 0.04 0.15674100000000002 rpy=0.0 -0.0 0.0 -> xyz=-0.08 0.04 0.15674100000000002 rpy=0.0 0.0 0.0
- joint part_6_hull_14_joint: origin xyz=-0.08 0.04 0.15674100000000002 rpy=0.0 -0.0 0.0 -> xyz=-0.08 0.04 0.15674100000000002 rpy=0.0 0.0 0.0
- joint part_6_hull_1_joint: origin xyz=-0.08 0.04 0.15674100000000002 rpy=0.0 -0.0 0.0 -> xyz=-0.08 0.04 0.15674100000000002 rpy=0.0 0.0 0.0
- joint part_6_hull_2_joint: origin xyz=-0.08 0.04 0.15674100000000002 rpy=0.0 -0.0 0.0 -> xyz=-0.08 0.04 0.15674100000000002 rpy=0.0 0.0 0.0
- joint part_6_hull_3_joint: origin xyz=-0.08 0.04 0.15674100000000002 rpy=0.0 -0.0 0.0 -> xyz=-0.08 0.04 0.15674100000000002 rpy=0.0 0.0 0.0
- joint part_6_hull_4_joint: origin xyz=-0.08 0.04 0.15674100000000002 rpy=0.0 -0.0 0.0 -> xyz=-0.08 0.04 0.15674100000000002 rpy=0.0 0.0 0.0
- joint part_6_hull_5_joint: origin xyz=-0.08 0.04 0.15674100000000002 rpy=0.0 -0.0 0.0 -> xyz=-0.08 0.04 0.15674100000000002 rpy=0.0 0.0 0.0
- joint part_6_hull_6_joint: origin xyz=-0.08 0.04 0.15674100000000002 rpy=0.0 -0.0 0.0 -> xyz=-0.08 0.04 0.15674100000000002 rpy=0.0 0.0 0.0
- joint part_6_hull_7_joint: origin xyz=-0.08 0.04 0.15674100000000002 rpy=0.0 -0.0 0.0 -> xyz=-0.08 0.04 0.15674100000000002 rpy=0.0 0.0 0.0
- joint part_6_hull_8_joint: origin xyz=-0.08 0.04 0.15674100000000002 rpy=0.0 -0.0 0.0 -> xyz=-0.08 0.04 0.15674100000000002 rpy=0.0 0.0 0.0
- joint part_6_hull_9_joint: origin xyz=-0.08 0.04 0.15674100000000002 rpy=0.0 -0.0 0.0 -> xyz=-0.08 0.04 0.15674100000000002 rpy=0.0 0.0 0.0

File: assets/urdf/fabrica/environments/beam_1/scene_sdf.urdf (robot description, URDF)
Before this commit: robot table_beam_1_scene_sdf, 5 links, 4 joints
Joints:
- joint part_2_joint: origin xyz=-0.124463 0.04 0.18810000000000004 rpy=3.141592653589793 -1.5707963267948966 3.141592653589793 -> xyz=-0.124463 0.04 0.18810000000000004 rpy=0.0 -1.5707963057214722 0.0
- joint part_3_joint: origin xyz=-0.035537 0.04 0.18810000000000004 rpy=3.141592653589793 -1.5707963267948966 3.141592653589793 -> xyz=-0.035537 0.04 0.18810000000000004 rpy=0.0 -1.5707963057214722 0.0
- joint part_6_joint: origin xyz=-0.08 0.04 0.15674100000000002 rpy=0.0 -0.0 0.0 -> xyz=-0.08 0.04 0.15674100000000002 rpy=0.0 0.0 0.0

File: assets/urdf/fabrica/environments/beam_2/scene.urdf (robot description, URDF)
Before this commit: robot table_beam_2_scene, 2 links, 1 joints
Joints:
- joint part_6_joint: origin xyz=-0.08 0.04 0.15674100000000002 rpy=0.0 -0.0 0.0 -> xyz=-0.08 0.04 0.15674100000000002 rpy=0.0 0.0 0.0

File: assets/urdf/fabrica/environments/beam_2/scene_coacd.urdf (robot description, URDF)
Before this commit: robot table_beam_2_scene_coacd, 16 links, 15 joints
Joints:
- joint part_6_hull_0_joint: origin xyz=-0.08 0.04 0.15674100000000002 rpy=0.0 -0.0 0.0 -> xyz=-0.08 0.04 0.15674100000000002 rpy=0.0 0.0 0.0
- joint part_6_hull_10_joint: origin xyz=-0.08 0.04 0.15674100000000002 rpy=0.0 -0.0 0.0 -> xyz=-0.08 0.04 0.15674100000000002 rpy=0.0 0.0 0.0
- joint part_6_hull_11_joint: origin xyz=-0.08 0.04 0.15674100000000002 rpy=0.0 -0.0 0.0 -> xyz=-0.08 0.04 0.15674100000000002 rpy=0.0 0.0 0.0
- joint part_6_hull_12_joint: origin xyz=-0.08 0.04 0.15674100000000002 rpy=0.0 -0.0 0.0 -> xyz=-0.08 0.04 0.15674100000000002 rpy=0.0 0.0 0.0
- joint part_6_hull_13_joint: origin xyz=-0.08 0.04 0.15674100000000002 rpy=0.0 -0.0 0.0 -> xyz=-0.08 0.04 0.15674100000000002 rpy=0.0 0.0 0.0
- joint part_6_hull_14_joint: origin xyz=-0.08 0.04 0.15674100000000002 rpy=0.0 -0.0 0.0 -> xyz=-0.08 0.04 0.15674100000000002 rpy=0.0 0.0 0.0
- joint part_6_hull_1_joint: origin xyz=-0.08 0.04 0.15674100000000002 rpy=0.0 -0.0 0.0 -> xyz=-0.08 0.04 0.15674100000000002 rpy=0.0 0.0 0.0
- joint part_6_hull_2_joint: origin xyz=-0.08 0.04 0.15674100000000002 rpy=0.0 -0.0 0.0 -> xyz=-0.08 0.04 0.15674100000000002 rpy=0.0 0.0 0.0
- joint part_6_hull_3_joint: origin xyz=-0.08 0.04 0.15674100000000002 rpy=0.0 -0.0 0.0 -> xyz=-0.08 0.04 0.15674100000000002 rpy=0.0 0.0 0.0
- joint part_6_hull_4_joint: origin xyz=-0.08 0.04 0.15674100000000002 rpy=0.0 -0.0 0.0 -> xyz=-0.08 0.04 0.15674100000000002 rpy=0.0 0.0 0.0
- joint part_6_hull_5_joint: origin xyz=-0.08 0.04 0.15674100000000002 rpy=0.0 -0.0 0.0 -> xyz=-0.08 0.04 0.15674100000000002 rpy=0.0 0.0 0.0
- joint part_6_hull_6_joint: origin xyz=-0.08 0.04 0.15674100000000002 rpy=0.0 -0.0 0.0 -> xyz=-0.08 0.04 0.15674100000000002 rpy=0.0 0.0 0.0
- joint part_6_hull_7_joint: origin xyz=-0.08 0.04 0.15674100000000002 rpy=0.0 -0.0 0.0 -> xyz=-0.08 0.04 0.15674100000000002 rpy=0.0 0.0 0.0
- joint part_6_hull_8_joint: origin xyz=-0.08 0.04 0.15674100000000002 rpy=0.0 -0.0 0.0 -> xyz=-0.08 0.04 0.15674100000000002 rpy=0.0 0.0 0.0
- joint part_6_hull_9_joint: origin xyz=-0.08 0.04 0.15674100000000002 rpy=0.0 -0.0 0.0 -> xyz=-0.08 0.04 0.15674100000000002 rpy=0.0 0.0 0.0

File: assets/urdf/fabrica/environments/beam_2/scene_sdf.urdf (robot description, URDF)
Before this commit: robot table_beam_2_scene_sdf, 2 links, 1 joints
Joints:
- joint part_6_joint: origin xyz=-0.08 0.04 0.15674100000000002 rpy=0.0 -0.0 0.0 -> xyz=-0.08 0.04 0.15674100000000002 rpy=0.0 0.0 0.0

File: assets/urdf/fabrica/environments/beam_3/scene.urdf (robot description, URDF)
Before this commit: robot table_beam_3_scene, 4 links, 3 joints
Joints:
- joint part_2_joint: origin xyz=-0.124463 0.04 0.18810000000000004 rpy=3.141592653589793 -1.5707963267948966 3.141592653589793 -> xyz=-0.124463 0.04 0.18810000000000004 rpy=0.0 -1.5707963057214722 0.0
- joint part_6_joint: origin xyz=-0.08 0.04 0.15674100000000002 rpy=0.0 -0.0 0.0 -> xyz=-0.08 0.04 0.15674100000000002 rpy=0.0 0.0 0.0
