Commit message: Add FabricaEnv with retract reward, optimize scene CoACD per adjacency
Phase 3 - FabricaEnv:
- New FabricaEnv class inheriting SimToolReal with retract-after-insertion
  reward: after all goals reached, robot is rewarded for retracting hand
  while object stays at final goal
- Retract reward gated on object remaining within final goal tolerance
- Successes clamped to prevent goal cycling during retract phase
- Config: enableRetract, retractRewardScale, retractDistanceThreshold,
  retractSuccessBonus
- Hydra configs: FabricaEnv.yaml, FabricaEnvLSTMAsymmetric.yaml + train

Scene CoACD optimization:
- Add inserts_into adjacency map to assembly_order.json
- generate_table_urdfs.py now only uses CoACD for the part being inserted
  into; other scene parts use raw mesh (single convex hull)
- Beam part 1 scene: 59 → 21 shapes (-64%)
- Beam part 3 scene: 42 → 15 shapes (-64%)
- Fixes OOM when training parts 1/3 at 24k envs on 48GB GPUs
- All insertion deltas verified < 1.2mm

Phase 2.6 experiment scripts for OOM retry (12k/24k variants)

Co-Authored-By: Claude Opus 4.6 (1M context) <noreply@anthropic.com>

File: assets/urdf/fabrica/environments/beam_0/scene_coacd.urdf (robot description, URDF)
Before this commit: robot table_beam_0_scene_coacd, 31 links, 30 joints
Links:
- removed link part_6_hull_0
- removed link part_6_hull_1
- removed link part_6_hull_10
- removed link part_6_hull_11
- removed link part_6_hull_2
- removed link part_6_hull_3
- removed link part_6_hull_4
- removed link part_6_hull_5
- removed link part_6_hull_6
- removed link part_6_hull_7
- removed link part_6_hull_8
- removed link part_6_hull_9
- added link part_6; collision mesh filename=../../beam/6/6_canonical.obj scale=1 1 1; visual mesh filename=../../beam/6/6_canonical.obj scale=1 1 1
Joints:
- removed joint part_6_hull_0_joint
- removed joint part_6_hull_10_joint
- removed joint part_6_hull_11_joint
- removed joint part_6_hull_1_joint
- removed joint part_6_hull_2_joint
- removed joint part_6_hull_3_joint
- removed joint part_6_hull_4_joint
- removed joint part_6_hull_5_joint
- removed joint part_6_hull_6_joint
- removed joint part_6_hull_7_joint
- removed joint part_6_hull_8_joint
- removed joint part_6_hull_9_joint
- added joint part_6_joint: type fixed, parent box, child part_6, origin xyz=-0.08 0.04 0.15674100000000002 rpy=0.0 0.0 0.0

File: assets/urdf/fabrica/environments/beam_1/scene_coacd.urdf (robot description, URDF)
Before this commit: robot table_beam_1_scene_coacd, 58 links, 57 joints
Links:
- removed link part_0_hull_0
- removed link part_0_hull_1
- removed link part_0_hull_2
- removed link part_0_hull_3
- removed link part_0_hull_4
- removed link part_0_hull_5
- removed link part_0_hull_6
- removed link part_0_hull_7
- removed link part_2_hull_0
- removed link part_2_hull_1
- removed link part_2_hull_10
- removed link part_2_hull_11
- removed link part_2_hull_12
- removed link part_2_hull_13
- removed link part_2_hull_14
- removed link part_2_hull_15
- removed link part_2_hull_16
- removed link part_2_hull_17
- removed link part_2_hull_2
- removed link part_2_hull_3
- removed link part_2_hull_4
- removed link part_2_hull_5
- removed link part_2_hull_6
- removed link part_2_hull_7
- removed link part_2_hull_8
- removed link part_2_hull_9
- removed link part_3_hull_17
- removed link part_3_hull_18
- removed link part_6_hull_0
- removed link part_6_hull_1
- removed link part_6_hull_10
- removed link part_6_hull_11
- removed link part_6_hull_2
- removed link part_6_hull_3
- removed link part_6_hull_4
- removed link part_6_hull_5
- removed link part_6_hull_6
- removed link part_6_hull_7
- removed link part_6_hull_8
- removed link part_6_hull_9
- added link part_0; collision mesh filename=../../beam/0/0_canonical.obj scale=1 1 1; visual mesh filename=../../beam/0/0_canonical.obj scale=1 1 1
- added link part_2; collision mesh filename=../../beam/2/2_canonical.obj scale=1 1 1; visual mesh filename=../../beam/2/2_canonical.obj scale=1 1 1
- added link part_6; collision mesh filename=../../beam/6/6_canonical.obj scale=1 1 1; visual mesh filename=../../beam/6/6_canonical.obj scale=1 1 1
- link part_3_hull_10: geometry collision mesh filename=../../beam/3/coacd/decomp_3.obj scale=1 1 1; visual mesh filename=../../beam/3/coacd/decomp_3.obj scale=1 1 1
- link part_3_hull_11: geometry collision mesh filename=../../beam/3/coacd/decomp_4.obj scale=1 1 1; visual mesh filename=../../beam/3/coacd/decomp_4.obj scale=1 1 1
- link part_3_hull_12: geometry collision mesh filename=../../beam/3/coacd/decomp_5.obj scale=1 1 1; visual mesh filename=../../beam/3/coacd/decomp_5.obj scale=1 1 1
- link part_3_hull_13: geometry collision mesh filename=../../beam/3/coacd/decomp_6.obj scale=1 1 1; visual mesh filename=../../beam/3/coacd/decomp_6.obj scale=1 1 1
- link part_3_hull_14: geometry collision mesh filename=../../beam/3/coacd/decomp_7.obj scale=1 1 1; visual mesh filename=../../beam/3/coacd/decomp_7.obj scale=1 1 1
- link part_3_hull_15: geometry collision mesh filename=../../beam/3/coacd/decomp_8.obj scale=1 1 1; visual mesh filename=../../beam/3/coacd/decomp_8.obj scale=1 1 1
- link part_3_hull_16: geometry collision mesh filename=../../beam/3/coacd/decomp_9.obj scale=1 1 1; visual mesh filename=../../beam/3/coacd/decomp_9.obj scale=1 1 1
- link part_3_hull_9: geometry collision mesh filename=../../beam/3/coacd/decomp_2.obj scale=1 1 1; visual mesh filename=../../beam/3/coacd/decomp_2.obj scale=1 1 1
Joints:
- removed joint part_0_hull_0_joint
- removed joint part_0_hull_1_joint
- removed joint part_0_hull_2_joint
- removed joint part_0_hull_3_joint
- removed joint part_0_hull_4_joint
- removed joint part_0_hull_5_joint
- removed joint part_0_hull_6_joint
- removed joint part_0_hull_7_joint
- removed joint part_2_hull_0_joint
- removed joint part_2_hull_10_joint
- removed joint part_2_hull_11_joint
- removed joint part_2_hull_12_joint
- removed joint part_2_hull_13_joint
- removed joint part_2_hull_14_joint
- removed joint part_2_hull_15_joint
- removed joint part_2_hull_16_joint
- removed joint part_2_hull_17_joint
- removed joint part_2_hull_1_joint
- removed joint part_2_hull_2_joint
- removed joint part_2_hull_3_joint
- removed joint part_2_hull_4_joint
- removed joint part_2_hull_5_joint
- removed joint part_2_hull_6_joint
- removed joint part_2_hull_7_joint
- removed joint part_2_hull_8_joint
- removed joint part_2_hull_9_joint
- removed joint part_3_hull_17_joint
- removed joint part_3_hull_18_joint
- removed joint part_6_hull_0_joint
- removed joint part_6_hull_10_joint
- removed joint part_6_hull_11_joint
- removed joint part_6_hull_1_joint
- removed joint part_6_hull_2_joint
- removed joint part_6_hull_3_joint
- removed joint part_6_hull_4_joint
- removed joint part_6_hull_5_joint
- removed joint part_6_hull_6_joint
- removed joint part_6_hull_7_joint
- removed joint part_6_hull_8_joint
- removed joint part_6_hull_9_joint
- added joint part_0_joint: type fixed, parent box, child part_0, origin xyz=-0.12445 0.04 0.22153 rpy=1.5707963267948966 0.0 -1.5707963267948966
- added joint part_2_joint: type fixed, parent box, child part_2, origin xyz=-0.124463 0.04 0.18810000000000004 rpy=0.0 -1.5707963057214722 0.0
- added joint part_6_joint: type fixed, parent box, child part_6, origin xyz=-0.08 0.04 0.15674100000000002 rpy=0.0 0.0 0.0

File: assets/urdf/fabrica/environments/beam_3/scene_coacd.urdf (robot description, URDF)
Before this commit: robot table_beam_3_scene_coacd, 39 links, 38 joints
Links:
- removed link part_0_hull_0
- removed link part_0_hull_1
- removed link part_0_hull_2
- removed link part_0_hull_3
- removed link part_0_hull_4
- removed link part_0_hull_5
- removed link part_0_hull_6
- removed link part_0_hull_7
- removed link part_2_hull_0
- removed link part_2_hull_1
- removed link part_2_hull_10
- removed link part_2_hull_11
- removed link part_2_hull_12
- removed link part_2_hull_13
- removed link part_2_hull_14
- removed link part_2_hull_15
- removed link part_2_hull_16
- removed link part_2_hull_17
- removed link part_2_hull_2
- removed link part_2_hull_3
- removed link part_2_hull_4
- removed link part_2_hull_5
- removed link part_2_hull_6
- removed link part_2_hull_7
- removed link part_2_hull_8
- removed link part_2_hull_9
- added link part_0; collision mesh filename=../../beam/0/0_canonical.obj scale=1 1 1; visual mesh filename=../../beam/0/0_canonical.obj scale=1 1 1
- added link part_2; collision mesh filename=../../beam/2/2_canonical.obj scale=1 1 1; visual mesh filename=../../beam/2/2_canonical.obj scale=1 1 1
Joints:
- removed joint part_0_hull_0_joint
- removed joint part_0_hull_1_joint
- removed joint part_0_hull_2_joint
- removed joint part_0_hull_3_joint
- removed joint part_0_hull_4_joint
- removed joint part_0_hull_5_joint
- removed joint part_0_hull_6_joint
- removed joint part_0_hull_7_joint
- removed joint part_2_hull_0_joint
- removed joint part_2_hull_10_joint
- removed joint part_2_hull_11_joint
- removed joint part_2_hull_12_joint
- removed joint part_2_hull_13_joint
- removed joint part_2_hull_14_joint
- removed joint part_2_hull_15_joint
- removed joint part_2_hull_16_joint
- removed joint part_2_hull_17_joint
- removed joint part_2_hull_1_joint
- removed joint part_2_hull_2_joint
- removed joint part_2_hull_3_joint
- removed joint part_2_hull_4_joint
- removed joint part_2_hull_5_joint
- removed joint part_2_hull_6_joint
- removed joint part_2_hull_7_joint
- removed joint part_2_hull_8_joint
- removed joint part_2_hull_9_joint
- added joint part_0_joint: type fixed, parent box, child part_0, origin xyz=-0.12445 0.04 0.22153 rpy=1.5707963267948966 0.0 -1.5707963267948966
- added joint part_2_joint: type fixed, parent box, child part_2, origin xyz=-0.124463 0.04 0.18810000000000004 rpy=0.0 -1.5707963057214722 0.0
