Commit message: Extend debug_insertion_training.py to all beam parts, fix part 6 CoACD
- Generalize debug_insertion_training.py with --assembly, --part, --method,
  --start-waypoint, --end-waypoint args (was hardcoded for part 2)
- Load trajectories dynamically from pick_place.json
- Auto-adjust camera to frame trajectory bounding box
- Include final timestep delta in video filename
- Increase max_gpu_contact_pairs to 16M (matching training fix)
- Re-run CoACD on part 6 with preprocess_resolution=100, resolution=8000
  to fix 3.9mm insertion collision for part 3 (now 0.6mm)
- Regenerate all scene_coacd.urdf files with updated part 6 hulls
- Add collision_comparison_summary.md documenting parameter tuning history

Co-Authored-By: Claude Opus 4.6 (1M context) <noreply@anthropic.com>

File: assets/urdf/fabrica/beam/6/coacd/beam_6_coacd.urdf (robot description, URDF)
Before this commit: robot beam_6_coacd, 16 links, 15 joints
Links:
- removed link hull_12
- removed link hull_13
- removed link hull_14
Joints:
- removed joint hull_joint_12
- removed joint hull_joint_13
- removed joint hull_joint_14

File: assets/urdf/fabrica/environments/beam_0/scene_coacd.urdf (robot description, URDF)
Before this commit: robot table_beam_0_scene_coacd, 34 links, 33 joints
Links:
- removed link part_6_hull_12
- removed link part_6_hull_13
- removed link part_6_hull_14
- link part_6_hull_10: geometry collision mesh filename=../../beam/6/coacd/decomp_8.obj scale=1 1 1; visual mesh filename=../../beam/6/coacd/decomp_8.obj scale=1 1 1
- link part_6_hull_11: geometry collision mesh filename=../../beam/6/coacd/decomp_9.obj scale=1 1 1; visual mesh filename=../../beam/6/coacd/decomp_9.obj scale=1 1 1
- link part_6_hull_4: geometry collision mesh filename=../../beam/6/coacd/decomp_2.obj scale=1 1 1; visual mesh filename=../../beam/6/coacd/decomp_2.obj scale=1 1 1
- link part_6_hull_5: geometry collision mesh filename=../../beam/6/coacd/decomp_3.obj scale=1 1 1; visual mesh filename=../../beam/6/coacd/decomp_3.obj scale=1 1 1
- link part_6_hull_6: geometry collision mesh filename=../../beam/6/coacd/decomp_4.obj scale=1 1 1; visual mesh filename=../../beam/6/coacd/decomp_4.obj scale=1 1 1
- link part_6_hull_7: geometry collision mesh filename=../../beam/6/coacd/decomp_5.obj scale=1 1 1; visual mesh filename=../../beam/6/coacd/decomp_5.obj scale=1 1 1
- link part_6_hull_8: geometry collision mesh filename=../../beam/6/coacd/decomp_6.obj scale=1 1 1; visual mesh filename=../../beam/6/coacd/decomp_6.obj scale=1 1 1
- link part_6_hull_9: geometry collision mesh filename=../../beam/6/coacd/decomp_7.obj scale=1 1 1; visual mesh filename=../../beam/6/coacd/decomp_7.obj scale=1 1 1
Joints:
- removed joint part_6_hull_12_joint
- removed joint part_6_hull_13_joint
- removed joint part_6_hull_14_joint

File: assets/urdf/fabrica/environments/beam_1/scene_coacd.urdf (robot description, URDF)
Before this commit: robot table_beam_1_scene_coacd, 59 links, 58 joints
Links:
- removed link part_6_hull_12
- removed link part_6_hull_13
- removed link part_6_hull_14
- added link part_3_hull_17; collision mesh filename=../../beam/3/coacd/decomp_8.obj scale=1 1 1; visual mesh filename=../../beam/3/coacd/decomp_8.obj scale=1 1 1
- added link part_3_hull_18; collision mesh filename=../../beam/3/coacd/decomp_9.obj scale=1 1 1; visual mesh filename=../../beam/3/coacd/decomp_9.obj scale=1 1 1
- link part_3_hull_10: geometry collision mesh filename=../../beam/3/coacd/decomp_18.obj scale=1 1 1; visual mesh filename=../../beam/3/coacd/decomp_18.obj scale=1 1 1
- link part_3_hull_11: geometry collision mesh filename=../../beam/3/coacd/decomp_2.obj scale=1 1 1; visual mesh filename=../../beam/3/coacd/decomp_2.obj scale=1 1 1
- link part_3_hull_12: geometry collision mesh filename=../../beam/3/coacd/decomp_3.obj scale=1 1 1; visual mesh filename=../../beam/3/coacd/decomp_3.obj scale=1 1 1
- link part_3_hull_13: geometry collision mesh filename=../../beam/3/coacd/decomp_4.obj scale=1 1 1; visual mesh filename=../../beam/3/coacd/decomp_4.obj scale=1 1 1
- link part_3_hull_14: geometry collision mesh filename=../../beam/3/coacd/decomp_5.obj scale=1 1 1; visual mesh filename=../../beam/3/coacd/decomp_5.obj scale=1 1 1
- link part_3_hull_15: geometry collision mesh filename=../../beam/3/coacd/decomp_6.obj scale=1 1 1; visual mesh filename=../../beam/3/coacd/decomp_6.obj scale=1 1 1
- link part_3_hull_16: geometry collision mesh filename=../../beam/3/coacd/decomp_7.obj scale=1 1 1; visual mesh filename=../../beam/3/coacd/decomp_7.obj scale=1 1 1
- link part_3_hull_9: geometry collision mesh filename=../../beam/3/coacd/decomp_17.obj scale=1 1 1; visual mesh filename=../../beam/3/coacd/decomp_17.obj scale=1 1 1
- link part_6_hull_10: geometry collision mesh filename=../../beam/6/coacd/decomp_8.obj scale=1 1 1; visual mesh filename=../../beam/6/coacd/decomp_8.obj scale=1 1 1
- link part_6_hull_11: geometry collision mesh filename=../../beam/6/coacd/decomp_9.obj scale=1 1 1; visual mesh filename=../../beam/6/coacd/decomp_9.obj scale=1 1 1
- link part_6_hull_4: geometry collision mesh filename=../../beam/6/coacd/decomp_2.obj scale=1 1 1; visual mesh filename=../../beam/6/coacd/decomp_2.obj scale=1 1 1
- link part_6_hull_5: geometry collision mesh filename=../../beam/6/coacd/decomp_3.obj scale=1 1 1; visual mesh filename=../../beam/6/coacd/decomp_3.obj scale=1 1 1
- link part_6_hull_6: geometry collision mesh filename=../../beam/6/coacd/decomp_4.obj scale=1 1 1; visual mesh filename=../../beam/6/coacd/decomp_4.obj scale=1 1 1
- link part_6_hull_7: geometry collision mesh filename=../../beam/6/coacd/decomp_5.obj scale=1 1 1; visual mesh filename=../../beam/6/coacd/decomp_5.obj scale=1 1 1
- link part_6_hull_8: geometry collision mesh filename=../../beam/6/coacd/decomp_6.obj scale=1 1 1; visual mesh filename=../../beam/6/coacd/decomp_6.obj scale=1 1 1
- link part_6_hull_9: geometry collision mesh filename=../../beam/6/coacd/decomp_7.obj scale=1 1 1; visual mesh filename=../../beam/6/coacd/decomp_7.obj scale=1 1 1
Joints:
- removed joint part_6_hull_12_joint
- removed joint part_6_hull_13_joint
- removed joint part_6_hull_14_joint
- added joint part_3_hull_17_joint: type fixed, parent box, child part_3_hull_17, origin xyz=-0.035537 0.04 0.18810000000000004 rpy=0.0 -1.5707963057214722 0.0
- added joint part_3_hull_18_joint: type fixed, parent box, child part_3_hull_18, origin xyz=-0.035537 0.04 0.18810000000000004 rpy=0.0 -1.5707963057214722 0.0

File: assets/urdf/fabrica/environments/beam_2/scene_coacd.urdf (robot description, URDF)
Before this commit: robot table_beam_2_scene_coacd, 16 links, 15 joints
Links:
- removed link part_6_hull_12
- removed link part_6_hull_13
- removed link part_6_hull_14
- link part_6_hull_10: geometry collision mesh filename=../../beam/6/coacd/decomp_8.obj scale=1 1 1; visual mesh filename=../../beam/6/coacd/decomp_8.obj scale=1 1 1
- link part_6_hull_11: geometry collision mesh filename=../../beam/6/coacd/decomp_9.obj scale=1 1 1; visual mesh filename=../../beam/6/coacd/decomp_9.obj scale=1 1 1
- link part_6_hull_4: geometry collision mesh filename=../../beam/6/coacd/decomp_2.obj scale=1 1 1; visual mesh filename=../../beam/6/coacd/decomp_2.obj scale=1 1 1
- link part_6_hull_5: geometry collision mesh filename=../../beam/6/coacd/decomp_3.obj scale=1 1 1; visual mesh filename=../../beam/6/coacd/decomp_3.obj scale=1 1 1
- link part_6_hull_6: geometry collision mesh filename=../../beam/6/coacd/decomp_4.obj scale=1 1 1; visual mesh filename=../../beam/6/coacd/decomp_4.obj scale=1 1 1
- link part_6_hull_7: geometry collision mesh filename=../../beam/6/coacd/decomp_5.obj scale=1 1 1; visual mesh filename=../../beam/6/coacd/decomp_5.obj scale=1 1 1
- link part_6_hull_8: geometry collision mesh filename=../../beam/6/coacd/decomp_6.obj scale=1 1 1; visual mesh filename=../../beam/6/coacd/decomp_6.obj scale=1 1 1
- link part_6_hull_9: geometry collision mesh filename=../../beam/6/coacd/decomp_7.obj scale=1 1 1; visual mesh filename=../../beam/6/coacd/decomp_7.obj scale=1 1 1
Joints:
- removed joint part_6_hull_12_joint
- removed joint part_6_hull_13_joint
- removed joint part_6_hull_14_joint

File: assets/urdf/fabrica/environments/beam_3/scene_coacd.urdf (robot description, URDF)
Before this commit: robot table_beam_3_scene_coacd, 42 links, 41 joints
Links:
- removed link part_6_hull_12
- removed link part_6_hull_13
- removed link part_6_hull_14
- link part_6_hull_10: geometry collision mesh filename=../../beam/6/coacd/decomp_8.obj scale=1 1 1; visual mesh filename=../../beam/6/coacd/decomp_8.obj scale=1 1 1
- link part_6_hull_11: geometry collision mesh filename=../../beam/6/coacd/decomp_9.obj scale=1 1 1; visual mesh filename=../../beam/6/coacd/decomp_9.obj scale=1 1 1
- link part_6_hull_4: geometry collision mesh filename=../../beam/6/coacd/decomp_2.obj scale=1 1 1; visual mesh filename=../../beam/6/coacd/decomp_2.obj scale=1 1 1
- link part_6_hull_5: geometry collision mesh filename=../../beam/6/coacd/decomp_3.obj scale=1 1 1; visual mesh filename=../../beam/6/coacd/decomp_3.obj scale=1 1 1
- link part_6_hull_6: geometry collision mesh filename=../../beam/6/coacd/decomp_4.obj scale=1 1 1; visual mesh filename=../../beam/6/coacd/decomp_4.obj scale=1 1 1
- link part_6_hull_7: geometry collision mesh filename=../../beam/6/coacd/decomp_5.obj scale=1 1 1; visual mesh filename=../../beam/6/coacd/decomp_5.obj scale=1 1 1
- link part_6_hull_8: geometry collision mesh filename=../../beam/6/coacd/decomp_6.obj scale=1 1 1; visual mesh filename=../../beam/6/coacd/decomp_6.obj scale=1 1 1
- link part_6_hull_9: geometry collision mesh filename=../../beam/6/coacd/decomp_7.obj scale=1 1 1; visual mesh filename=../../beam/6/coacd/decomp_7.obj scale=1 1 1
Joints:
- removed joint part_6_hull_12_joint
- removed joint part_6_hull_13_joint
- removed joint part_6_hull_14_joint
