Commit message: Reorganize benchmark_processing pipeline and clean up fabrica/
- Rename step scripts to match pipeline order (step0-6)
- Add --viz to all processing scripts (viser viewers)
- Create step1_define_assembly_order.py (interactive UI)
- Create step6_validate_insertions.py (IsaacGym teleport-test)
- Simplify all scripts (step0: 229→120, step2: 457→197, step3: 680→280 lines)
- Add CoACD overshoot metric to step4
- Add collision method toggle (coacd/sdf/vhacd) to step5 viz
- Move trajectories into assets/urdf/fabrica/{assembly}/trajectories/
- Move environments into assets/urdf/fabrica/{assembly}/environments/
- Update all path references (fabrica_env, fabrica_eval, isaacsim_conversion)
- Delete absorbed viz/debug scripts from fabrica/
- Delete redundant eval scripts (keep only fabrica_eval.py)
- Consolidate train_scripts into experiments/
- Update baseline.sub to unified multi-part training with retract
- Rewrite fabrica_setup.md and README.md
- Add fabrica_example and trajectories_example to .gitignore

Co-Authored-By: Claude Opus 4.6 (1M context) <noreply@anthropic.com>

File: assets/urdf/fabrica/beam/1/coacd/beam_1_coacd.urdf (robot description, URDF)
Before this commit: robot beam_1_coacd, 9 links, 8 joints
Links:
- removed link hull_7
Joints:
- removed joint hull_joint_7

File: assets/urdf/fabrica/beam/2/coacd/beam_2_coacd.urdf (robot description, URDF)
Before this commit: robot beam_2_coacd, 19 links, 18 joints
Links:
- removed link hull_17
Joints:
- removed joint hull_joint_17

File: assets/urdf/fabrica/beam/3/coacd/beam_3_coacd.urdf (robot description, URDF)
Before this commit: robot beam_3_coacd, 18 links, 17 joints
Links:
- removed link hull_12
- removed link hull_13
- removed link hull_14
- removed link hull_15
- removed link hull_16
Joints:
- removed joint hull_joint_12
- removed joint hull_joint_13
- removed joint hull_joint_14
- removed joint hull_joint_15
- removed joint hull_joint_16

File: assets/urdf/fabrica/beam/6/coacd/beam_6_coacd.urdf (robot description, URDF)
Before this commit: robot beam_6_coacd, 13 links, 12 joints
Links:
- added link hull_12, mass 0.001; collision mesh filename=decomp_12.obj scale=1 1 1; visual mesh filename=decomp_12.obj scale=1 1 1
- added link hull_13, mass 0.001; collision mesh filename=decomp_13.obj scale=1 1 1; visual mesh filename=decomp_13.obj scale=1 1 1
- added link hull_14, mass 0.001; collision mesh filename=decomp_14.obj scale=1 1 1; visual mesh filename=decomp_14.obj scale=1 1 1
Joints:
- added joint hull_joint_12: type fixed, parent base_link, child hull_12, origin xyz=0 0 0 rpy=0 0 0
- added joint hull_joint_13: type fixed, parent base_link, child hull_13, origin xyz=0 0 0 rpy=0 0 0
- added joint hull_joint_14: type fixed, parent base_link, child hull_14, origin xyz=0 0 0 rpy=0 0 0
