Commit message: Re-run beam CoACD with seed 2 and generalize sweep script
- Regenerate beam CoACD decompositions using seed 2, which passes
  all insertion validation tests (worst: part 1 at 2.2mm pos, 2.5mm kp)
- Update scene_coacd URDFs to match new decomposition counts
- Generalize sweep_coacd_seeds.py to work for any assembly:
  - Add --assembly arg (replaces hardcoded car)
  - Auto-detect parts from assembly_order.json
  - Decompose all parts per seed (not just insertion targets)
  - Parallelize step4 and step6 within each seed
  - Add --max-seeds, --max-pos, --max-kp, --coacd-args flags
- Fix .gitignore to match isaacgym symlink

Co-Authored-By: Claude Opus 4.6 (1M context) <noreply@anthropic.com>

File: assets/urdf/fabrica/beam/0/coacd/beam_0_coacd.urdf (robot description, URDF)
Before this commit: robot beam_0_coacd, 9 links, 8 joints
Links:
- removed link hull_6
- removed link hull_7
Joints:
- removed joint hull_joint_6
- removed joint hull_joint_7

File: assets/urdf/fabrica/beam/1/coacd/beam_1_coacd.urdf (robot description, URDF)
Before this commit: robot beam_1_coacd, 8 links, 7 joints
Links:
- added link hull_7, mass 0.001; collision mesh filename=decomp_7.obj scale=1 1 1; visual mesh filename=decomp_7.obj scale=1 1 1
Joints:
- added joint hull_joint_7: type fixed, parent base_link, child hull_7, origin xyz=0 0 0 rpy=0 0 0

File: assets/urdf/fabrica/beam/2/coacd/beam_2_coacd.urdf (robot description, URDF)
Before this commit: robot beam_2_coacd, 18 links, 17 joints
Links:
- removed link hull_16
Joints:
- removed joint hull_joint_16

File: assets/urdf/fabrica/beam/3/coacd/beam_3_coacd.urdf (robot description, URDF)
Before this commit: robot beam_3_coacd, 13 links, 12 joints
Links:
- added link hull_12, mass 0.001; collision mesh filename=decomp_12.obj scale=1 1 1; visual mesh filename=decomp_12.obj scale=1 1 1
Joints:
- added joint hull_joint_12: type fixed, parent base_link, child hull_12, origin xyz=0 0 0 rpy=0 0 0

File: assets/urdf/fabrica/beam/6/coacd/beam_6_coacd.urdf (robot description, URDF)
Before this commit: robot beam_6_coacd, 16 links, 15 joints
Links:
- removed link hull_14
Joints:
- removed joint hull_joint_14

File: assets/urdf/fabrica/beam/environments/0/scene_coacd.urdf (robot description, URDF)
Before this commit: robot table_beam_0_scene_coacd, 19 links, 18 joints
Links:
- removed link part_2_hull_16
- link part_2_hull_10: geometry collision mesh filename=../../2/coacd/decomp_4.obj scale=1 1 1; visual mesh filename=../../2/coacd/decomp_4.obj scale=1 1 1
- link part_2_hull_11: geometry collision mesh filename=../../2/coacd/decomp_5.obj scale=1 1 1; visual mesh filename=../../2/coacd/decomp_5.obj scale=1 1 1
- link part_2_hull_12: geometry collision mesh filename=../../2/coacd/decomp_6.obj scale=1 1 1; visual mesh filename=../../2/coacd/decomp_6.obj scale=1 1 1
- link part_2_hull_13: geometry collision mesh filename=../../2/coacd/decomp_7.obj scale=1 1 1; visual mesh filename=../../2/coacd/decomp_7.obj scale=1 1 1
- link part_2_hull_14: geometry collision mesh filename=../../2/coacd/decomp_8.obj scale=1 1 1; visual mesh filename=../../2/coacd/decomp_8.obj scale=1 1 1
- link part_2_hull_15: geometry collision mesh filename=../../2/coacd/decomp_9.obj scale=1 1 1; visual mesh filename=../../2/coacd/decomp_9.obj scale=1 1 1
- link part_2_hull_8: geometry collision mesh filename=../../2/coacd/decomp_2.obj scale=1 1 1; visual mesh filename=../../2/coacd/decomp_2.obj scale=1 1 1
- link part_2_hull_9: geometry collision mesh filename=../../2/coacd/decomp_3.obj scale=1 1 1; visual mesh filename=../../2/coacd/decomp_3.obj scale=1 1 1
Joints:
- removed joint part_2_hull_16_joint

File: assets/urdf/fabrica/beam/environments/1/scene_coacd.urdf (robot description, URDF)
Before this commit: robot table_beam_1_scene_coacd, 16 links, 15 joints
Links:
- added link part_3_hull_12; collision mesh filename=../../3/coacd/decomp_9.obj scale=1 1 1; visual mesh filename=../../3/coacd/decomp_9.obj scale=1 1 1
- link part_3_hull_10: geometry collision mesh filename=../../3/coacd/decomp_7.obj scale=1 1 1; visual mesh filename=../../3/coacd/decomp_7.obj scale=1 1 1
- link part_3_hull_11: geometry collision mesh filename=../../3/coacd/decomp_8.obj scale=1 1 1; visual mesh filename=../../3/coacd/decomp_8.obj scale=1 1 1
- link part_3_hull_4: geometry collision mesh filename=../../3/coacd/decomp_12.obj scale=1 1 1; visual mesh filename=../../3/coacd/decomp_12.obj scale=1 1 1
- link part_3_hull_5: geometry collision mesh filename=../../3/coacd/decomp_2.obj scale=1 1 1; visual mesh filename=../../3/coacd/decomp_2.obj scale=1 1 1
- link part_3_hull_6: geometry collision mesh filename=../../3/coacd/decomp_3.obj scale=1 1 1; visual mesh filename=../../3/coacd/decomp_3.obj scale=1 1 1
- link part_3_hull_7: geometry collision mesh filename=../../3/coacd/decomp_4.obj scale=1 1 1; visual mesh filename=../../3/coacd/decomp_4.obj scale=1 1 1
- link part_3_hull_8: geometry collision mesh filename=../../3/coacd/decomp_5.obj scale=1 1 1; visual mesh filename=../../3/coacd/decomp_5.obj scale=1 1 1
- link part_3_hull_9: geometry collision mesh filename=../../3/coacd/decomp_6.obj scale=1 1 1; visual mesh filename=../../3/coacd/decomp_6.obj scale=1 1 1
Joints:
- added joint part_3_hull_12_joint: type fixed, parent box, child part_3_hull_12, origin xyz=-0.035537 0.04 0.18770900000000001 rpy=0.0 -1.5707963057214722 0.0

File: assets/urdf/fabrica/beam/environments/2/scene_coacd.urdf (robot description, URDF)
Before this commit: robot table_beam_2_scene_coacd, 16 links, 15 joints
Links:
- removed link part_6_hull_14
- link part_6_hull_10: geometry collision mesh filename=../../6/coacd/decomp_6.obj scale=1 1 1; visual mesh filename=../../6/coacd/decomp_6.obj scale=1 1 1
- link part_6_hull_11: geometry collision mesh filename=../../6/coacd/decomp_7.obj scale=1 1 1; visual mesh filename=../../6/coacd/decomp_7.obj scale=1 1 1
- link part_6_hull_12: geometry collision mesh filename=../../6/coacd/decomp_8.obj scale=1 1 1; visual mesh filename=../../6/coacd/decomp_8.obj scale=1 1 1
- link part_6_hull_13: geometry collision mesh filename=../../6/coacd/decomp_9.obj scale=1 1 1; visual mesh filename=../../6/coacd/decomp_9.obj scale=1 1 1
- link part_6_hull_6: geometry collision mesh filename=../../6/coacd/decomp_2.obj scale=1 1 1; visual mesh filename=../../6/coacd/decomp_2.obj scale=1 1 1
- link part_6_hull_7: geometry collision mesh filename=../../6/coacd/decomp_3.obj scale=1 1 1; visual mesh filename=../../6/coacd/decomp_3.obj scale=1 1 1
- link part_6_hull_8: geometry collision mesh filename=../../6/coacd/decomp_4.obj scale=1 1 1; visual mesh filename=../../6/coacd/decomp_4.obj scale=1 1 1
- link part_6_hull_9: geometry collision mesh filename=../../6/coacd/decomp_5.obj scale=1 1 1; visual mesh filename=../../6/coacd/decomp_5.obj scale=1 1 1
Joints:
- removed joint part_6_hull_14_joint

File: assets/urdf/fabrica/beam/environments/3/scene_coacd.urdf (robot description, URDF)
Before this commit: robot table_beam_3_scene_coacd, 18 links, 17 joints
Links:
- removed link part_6_hull_14
- link part_6_hull_10: geometry collision mesh filename=../../6/coacd/decomp_6.obj scale=1 1 1; visual mesh filename=../../6/coacd/decomp_6.obj scale=1 1 1
- link part_6_hull_11: geometry collision mesh filename=../../6/coacd/decomp_7.obj scale=1 1 1; visual mesh filename=../../6/coacd/decomp_7.obj scale=1 1 1
- link part_6_hull_12: geometry collision mesh filename=../../6/coacd/decomp_8.obj scale=1 1 1; visual mesh filename=../../6/coacd/decomp_8.obj scale=1 1 1
- link part_6_hull_13: geometry collision mesh filename=../../6/coacd/decomp_9.obj scale=1 1 1; visual mesh filename=../../6/coacd/decomp_9.obj scale=1 1 1
- link part_6_hull_6: geometry collision mesh filename=../../6/coacd/decomp_2.obj scale=1 1 1; visual mesh filename=../../6/coacd/decomp_2.obj scale=1 1 1
- link part_6_hull_7: geometry collision mesh filename=../../6/coacd/decomp_3.obj scale=1 1 1; visual mesh filename=../../6/coacd/decomp_3.obj scale=1 1 1
- link part_6_hull_8: geometry collision mesh filename=../../6/coacd/decomp_4.obj scale=1 1 1; visual mesh filename=../../6/coacd/decomp_4.obj scale=1 1 1
- link part_6_hull_9: geometry collision mesh filename=../../6/coacd/decomp_5.obj scale=1 1 1; visual mesh filename=../../6/coacd/decomp_5.obj scale=1 1 1
Joints:
- removed joint part_6_hull_14_joint
