Commit message: non-bolted fixture: dynamic receptive + fixture-tracking goal observation
Reviewer-requested setup: evaluate existing policies against a fixture that
isn't bolted down, with no retraining.

env (peg_in_hole):
- new `peg_in_hole.fixture_bolted` (default True). When False the receptive is
  baked as a dynamic rigid body (kinematic/gravity flags flipped) instead of a
  kinematic one, so the peg can push it. The bolted branch keeps the original
  prop set byte-for-byte -- max_depenetration_velocity is added only in the
  dynamic case -- so the default path is unchanged.
- `_refresh_free_fixture_goal()` re-derives the insertion goal from the
  fixture's live pose every step. hole_pos/hole_quat_wxyz were previously
  written at reset and never read back, and the goal was only rewritten on
  subgoal transitions, so both went stale the instant the fixture moved. It
  rewrites goal_viz -- which is what the policy observes (obs_utils reads
  goal_viz.data.root_pos_w) -- so the observation layout is unchanged and the
  policy needs no retraining. Restricted to non-random-goal envs (random-goal
  envs park the hole at a z=-1 sentinel) in the tail phase.
- `_write_goal_pose(subgoal_override=...)`: the internal
  `_successes % env_max_goals` wraps a completed env back to subgoal 0, which
  yanked the goal marker from final-insert back to pre-insert the moment
  insertion landed (and would have broken retract, judged against goal_viz).
  The refresh now clamps instead, pinning a completed env to the final
  insertion pose while still tracking the fixture.

assets: the four insertion fixtures carried mass properties that were dead
weight while kinematic -- the peg hole had 10 kg / I=0.1 / a COM above the part,
and the beam and furniture fixtures had no <inertial> at all (importer default).
A 10 kg block barely responds to peg contact. New scripts/compute_urdf_inertial.py
derives mass, COM and the full inertia tensor from the collision geometry at a
material density (boxes with rpy rotation + trimesh for meshes, combined by
parallel axis); validated against a hand computation of the peg hole. At solid
PLA: peg hole 0.436 kg, beam p0 0.690 kg, beam p2 0.383 kg, furniture 0.280 kg.
NOTE: the furniture receptive is a hollow shell (5 mm plate + rim walls), so its
225.6 cm^3 is deposited-material volume, not the 825 cm^3 solid part -- 0.280 kg
corresponds to a ~27%-infill print rather than a solid top.

tooling:
- offline_eval_obj_pose_noise_sweep.py: --hold-xyz / --hold-rot to freeze one
  axis at its training value and sweep the other, isolating which one drives
  the collapse (a joint sweep cannot attribute it).
- plot_noise_sweep.py: N series via repeated --json/--label, legend for >=2
  series, data-driven axis limits so partial sweeps render correctly.
- plot_fixture_bars.py: bolted vs unbolted grouped bars.

First numbers (peg, 512 envs, 1 episode/env, no early drops):
bolted 98.02% -> unbolted 88.44%.

Co-Authored-By: Claude Opus 5 <noreply@anthropic.com>
Claude-Session: https://claude.ai/code/session_01FWKYPNDkZivptTjPibs2A9

File: assets/urdf/fabrica/beam_3x/insertion_fixtures/part_0_sdf_hybrid.urdf (robot description, URDF)
Before this commit: robot fixture_beam_3x_part_0_sdf_hybrid, 1 links, 0 joints
Links:
- link plate: mass None -> 0.6898

File: assets/urdf/fabrica/beam_3x/insertion_fixtures/part_2_sdf_hybrid.urdf (robot description, URDF)
Before this commit: robot fixture_beam_3x_part_2_sdf_hybrid, 1 links, 0 joints
Links:
- link plate: mass None -> 0.3826

File: assets/urdf/furniture_bench/square_table/insertion_fixtures/one_leg_sdf_hybrid.urdf (robot description, URDF)
Before this commit: robot one_leg_receptive_sdf_hybrid, 1 links, 0 joints
Links:
- link receptive: mass None -> 0.2798
