Commit message: one_leg fixture: mass 0.2798 -> 0.6001 kg
The old value came from shell volume, which is meaningless while the fixture is
kinematic -- PhysX ignores mass properties entirely for bolted fixtures. It
starts to matter once peg_in_hole.fixture_bolted=False makes the receptive
dynamic, where 0.28 kg let the table top slide off the table during screwing.

Recomputed from the collision geometry as a solid at the same density; the
inertia tensor is rescaled to match.

Co-Authored-By: Claude Opus 5 <noreply@anthropic.com>
Claude-Session: https://claude.ai/code/session_01FWKYPNDkZivptTjPibs2A9

File: assets/urdf/furniture_bench/square_table/insertion_fixtures/one_leg_sdf_hybrid.urdf (robot description, URDF)
Before this commit: robot one_leg_receptive_sdf_hybrid, 1 links, 0 joints
Links:
- link receptive: mass 0.2798 -> 0.6001
