Commit message: plug_fork: fix socket collision depth, plug visual frame, holder material
Three defects in the generated assets, all invisible to the checks that were
running -- extents matched, URDFs parsed, success rates climbed.

Socket collision was a solid 120x56x26 mm block with a 4 mm slot, against
15.9 mm blades, so the plug seated 11.9 mm proud and still scored success.
Rebuilt as floor + four cavity walls + a slotted face with the cavity opened
to the full blade length. create_assets.py held a duplicate copy of the box
layout, which is why the first fix silently did nothing; it now calls the
authoritative socket_collision_boxes() in viz_insertion_spec.

plug_visual.glb was 90 degrees off its own collision boxes -- prongs along Z
in the visual, along X in collision. Scene.apply_transform only sets a node
transform and it did not survive the GLB round-trip, while the collision
boxes were rotated explicitly. The rotation is now baked into the vertices.

The holder exported a bare OBJ, which carries no material, so viewers drew it
solid black. It now gets a stainless PBR material and exports GLB, matching
what the plug and socket already did.

Co-Authored-By: Claude Opus 5 (1M context) <noreply@anthropic.com>
Claude-Session: https://claude.ai/code/session_01FWKYPNDkZivptTjPibs2A9

File: assets/urdf/plug_fork/holder/holder_tol0p5mm.urdf (robot description, URDF)
Before this commit: robot holder_tol0p5mm, 1 links, 0 joints
Links:
- link hole: geometry collision box size=0.016434 0.025154 0.080000; collision box size=0.016434 0.025154 0.080000

File: assets/urdf/plug_fork/holder/holder_tol1mm.urdf (robot description, URDF)
Before this commit: robot holder_tol1mm, 1 links, 0 joints
Links:
- link hole: geometry collision box size=0.017434 0.024654 0.080000; collision box size=0.017434 0.024654 0.080000

File: assets/urdf/plug_fork/holder/holder_tol2mm.urdf (robot description, URDF)
Before this commit: robot holder_tol2mm, 1 links, 0 joints
Links:
- link hole: geometry collision box size=0.019434 0.023654 0.080000; collision box size=0.019434 0.023654 0.080000

File: assets/urdf/plug_fork/socket/socket_tol0p1mm.urdf (robot description, URDF)
Before this commit: robot socket_tol0p1mm, 1 links, 0 joints
Links:
- link hole: mass 0.302236 -> 0.290976; geometry collision box size=0.001800 0.023800 0.004000; collision box size=0.001800 0.023800 0.004000

File: assets/urdf/plug_fork/socket/socket_tol0p3mm.urdf (robot description, URDF)
Before this commit: robot socket_tol0p3mm, 1 links, 0 joints
Links:
- link hole: mass 0.302189 -> 0.290460; geometry collision box size=0.002200 0.023600 0.004000; collision box size=0.002200 0.023600 0.004000

File: assets/urdf/plug_fork/socket/socket_tol0p5mm.urdf (robot description, URDF)
Before this commit: robot socket_tol0p5mm, 1 links, 0 joints
Links:
- link hole: mass 0.302138 -> 0.289930; geometry collision box size=0.002600 0.023400 0.004000; collision box size=0.002600 0.023400 0.004000

File: assets/urdf/plug_fork/socket/socket_tol1mm.urdf (robot description, URDF)
Before this commit: robot socket_tol1mm, 1 links, 0 joints
Links:
- link hole: mass 0.301994 -> 0.288548; geometry collision box size=0.003600 0.022900 0.004000; collision box size=0.003600 0.022900 0.004000
